File: pmod_sfp/pmod_sfp.kicad_sch (KiCad schematic)
At the start: 3 parts, among them J1 SFP, U1 Pmod_connector

Commit message: Almost ended board
Parts:
- added C1: 22uF, Capacitor_SMD:C_0402_1005Metric, symbol Device:C
- added C2, C4, C6: 0.1uF, Capacitor_SMD:C_0402_1005Metric, symbol Device:C
- added C3, C5: 10uF, Capacitor_SMD:C_0402_1005Metric, symbol Device:C
- added L1, L2: 220@100MHz, Inductor_SMD:L_0402_1005Metric, symbol Device:L_Iron
- added R2, R3: 4.7k, Resistor_SMD:R_0402_1005Metric, symbol Device:R_US
Connections:
- net +3V3: now also C1.1, C2.1, L1.1, L2.1, R2.1, R3.2
- net GND: now also C1.2, C2.2, C3.2, C4.2, C5.2, C6.2
- net SFP_LOSS: now also R3.1
- net SFP_TX_DIS: now also R2.2
- net at J1.15 (VccR): now also C5.1, C6.1, L2.2
- net at J1.16 (VccT): now also C3.1, C4.1, L1.2

Commit message: update
Parts:
- U1: footprint Pmod:DIP-12_100 -> Pmod:PMOD_EXTENSION_BOARD
Changed lines of the file:
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@@
     (property "Reference" "U1" (id 0) (at 67.31 57.15 0))
     (property "Value" "Pmod_connector" (id 1) (at 67.31 59.69 0))
-    (property "Footprint" "Pmod:DIP-12_100" (id 2) (at 74.93 83.82 0)
+    (property "Footprint" "Pmod:PMOD_EXTENSION_BOARD" (id 2) (at 74.93 83.82 0)
       (effects (font (size 1.27 1.27)) hide)
     )
@@
     )
     (path "/dd689124-b5c5-4dc7-813d-a0bf1f8a781e"
-      (reference "U1") (unit 1) (value "Pmod_connector") (footprint "Pmod:DIP-12_100")
+      (reference "U1") (unit 1) (value "Pmod_connector") (footprint "Pmod:PMOD_EXTENSION_BOARD")
     )
   )
