File: pmod_sfp/pmod_sfp.kicad_pcb (KiCad board)
At the start: 2 copper layers, 69.1 x 20.3 mm, 3 parts, among them J1 SFP, U1 Pmod_connector

Commit message: Almost ended board
Parts:
- added C1: 22uF, Capacitor_SMD:C_0402_1005Metric, F.Cu at (162.0, 64.3)
- added C2: 0.1uF, Capacitor_SMD:C_0402_1005Metric, F.Cu at (162.1, 63.0)
- added C3: 10uF, Capacitor_SMD:C_0402_1005Metric, F.Cu at (168.9, 67.8)
- added C4: 0.1uF, Capacitor_SMD:C_0402_1005Metric, F.Cu at (168.9, 66.5)
- added C5: 10uF, Capacitor_SMD:C_0402_1005Metric, F.Cu at (168.9, 69.1)
- added C6: 0.1uF, Capacitor_SMD:C_0402_1005Metric, F.Cu at (168.9, 70.4)
- added L1: 220@100MHz, Inductor_SMD:L_0402_1005Metric, F.Cu at (168.9, 65.3)
- added L2: 220@100MHz, Inductor_SMD:L_0402_1005Metric, F.Cu at (168.9, 64.0)
- added R2: 4.7k, Resistor_SMD:R_0402_1005Metric, F.Cu at (162.1, 70.1)
- added R3: 4.7k, Resistor_SMD:R_0402_1005Metric, F.Cu at (162.1, 68.6)
- moved R1 3.81 mm to (162.1, 67.1), turned to 180 degrees
Connections:
- J1 pad 15: unconnected-(J1-Pad15) -> Net-(J1-Pad15)
- J1 pad 16: unconnected-(J1-Pad16) -> Net-(C3-Pad1)
Routing:
- net GND: track 0.00 -> 50.5 mm, vias 0 -> 8
- net +3V3: track 0.00 -> 43.0 mm
- net /SFP_LOSS: track 0.00 -> 42.0 mm, vias 0 -> 2
- net Net-(J1-Pad15): track 0.00 -> 38.9 mm, vias 0 -> 2
- net /SFP_TX_DIS: track 0.00 -> 37.7 mm, vias 0 -> 2
- net Net-(C3-Pad1): track 0.00 -> 35.4 mm, vias 0 -> 2
- net /SFP_RX_P: track 0.00 -> 27.5 mm
- net /SFP_RX_N: track 0.00 -> 26.8 mm
- net /SFP_TX_P: track 0.00 -> 26.2 mm, vias 0 -> 1
- net /SFP_TX_N: track 0.00 -> 25.4 mm, vias 0 -> 1
- net Net-(J1-Pad7): track 0.00 -> 22.2 mm, vias 0 -> 2
- added copper zone on B.Cu, net GND

Commit message: update
Parts:
- U1: footprint Pmod:DIP-12_100 -> Pmod:PMOD_EXTENSION_BOARD
- moved U1 0.26 mm to (175.0, 71.0), turned to 90 degrees
Other:
- board text added: "https://github.com/DRubioG/pmod_sfp"
Changed lines of the file:
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@@
   (net 11 "/SFP_TX_P")
   (net 12 "Net-(C3-Pad1)")
-  (net 13 "Net-(J1-Pad15)")
+  (net 13 "Net-(C5-Pad1)")
   (net 14 "/SFP_TX_N")
   (net 15 "+3V3")
@@
     )
   )
-  (footprint "Pmod:DIP-12_100" (layer "F.Cu")
-    (at 175.24 71.12 -90)
-    (property "Sheetfile" "pmod_sfp.kicad_sch")
-    (property "Sheetname" "")
-    (fp_text reference "U1" (at -8.85 0) (layer "F.SilkS")
-      (effects (font (size 1 1) (thickness 0.15)))
-    )
-    (fp_text value "Pmod_connector" (at 0 0 90) (layer "F.Fab")
-      (effects (font (size 1 1) (thickness 0.15)))
-    )
-    (fp_line (start 1.85 2.8) (end 7.85 2.77) (layer "F.SilkS") (width 0.12))
-    (fp_line (start -7.49 -0.923333) (end -7.49 0.923333) (layer "F.SilkS") (width 0.12))
-    (fp_line (start 7.85 2.77) (end 7.85 -2.769999) (layer "F.SilkS") (width 0.12))
-    (fp_line (start -2.35 2.8) (end -7.85 2.769999) (layer "F.SilkS") (width 0.12))
-    (fp_line (start 7.85 -2.769999) (end -7.85 -2.77) (layer "F.SilkS") (width 0.12))
-    (fp_line (start -7.85 -0.923333) (end -7.49 -0.923333) (layer "F.SilkS") (width 0.12))
-    (fp_line (start -7.85 -2.77) (end -7.85 -0.923333) (layer "F.SilkS") (width 0.12))
-    (fp_line (start 1.85 3.4) (end 1.85 2.8) (layer "F.SilkS") (width 0.12))
-    (fp_line (start -2.3 2.8) (end -2.3 3.4) (layer "F.SilkS") (width 0.12))
-    (fp_line (start -2.3 3.4) (end 1.85 3.4) (layer "F.SilkS") (width 0.12))
-    (fp_line (start -7.49 0.923333) (end -7.85 0.923333) (layer "F.SilkS") (width 0.12))
-    (fp_line (start -7.85 0.923333) (end -7.85 2.769999) (layer "F.SilkS") (width 0.12))
-    (fp_line (start 7.6 -2.52) (end 7.6 2.52) (layer "F.CrtYd") (width 0.05))
-    (fp_line (start -7.6 2.52) (end -7.6 -2.52) (layer "F.CrtYd") (width 0.05))
-    (fp_line (start 7.6 2.52) (end -7.6 2.52) (layer "F.CrtYd") (width 0.05))
-    (fp_line (start -7.6 -2.52) (end 7.6 -2.52) (layer "F.CrtYd") (width 0.05))
-    (pad "1" thru_hole rect (at -6.35 1.27 270) (size 1.5 1.5) (drill 0.8) (layers *.Cu *.Mask)
+  (footprint "Pmod:PMOD_EXTENSION_BOARD" (layer "F.Cu")
+    (at 174.99 71.05 90)
+    (descr "This PMOD goes in the extension board")
+    (property "Sheetfile" "pmod_sfp.kicad_sch")
+    (property "Sheetname" "")
+    (fp_text reference "U1" (at 9.6 0) (layer "F.SilkS")
+      (effects (font (size 1 1) (thickness 0.15)))
+    )
+    (fp_text value "Pmod_connector" (at 0 4.6 90) (layer "F.Fab")
+      (effects (font (size 1 1) (thickness 0.15)))
+    )
+    (fp_text user "GND" (at 3.8 -4.2 180 unlocked) (layer "F.SilkS")
+      (effects (font (size 1 1) (thickness 0.15)))
+    )
+    (fp_text user "VCC" (at 6.4 -4.2 180 unlocked) (layer "F.SilkS")
+      (effects (font (size 1 1) (thickness 0.15)))
+    )
+    (fp_line (start 2.23 -3.13) (end -1.92 -3.13) (layer "F.SilkS") (width 0.12))
+    (fp_line (start 2.23 -2.5) (end 2.23 -3.13) (layer "F.SilkS") (width 0.12))
+    (fp_line (start -7.92 -2.5) (end -7.92 3.039999) (layer "F.SilkS") (width 0.12))
+    (fp_line (start 2.23 -2.5) (end 7.73 -2.5) (layer "F.SilkS") (width 0.12))
+    (fp_line (start 7.78 -0.653333) (end 7.78 -2.499999) (layer "F.SilkS") (width 0.12))
+    (fp_line (start 7.78 1.193333) (end 7.42 1.193333) (layer "F.SilkS") (width 0.12))
+    (fp_line (start 7.42 -0.653333) (end 7.78 -0.653333) (layer "F.SilkS") (width 0.12))
+    (fp_line (start -7.92 3.039999) (end 7.78 3.04) (layer "F.SilkS") (width 0.12))
+    (fp_line (start -1.92 -3.13) (end -1.92 -2.5) (layer "F.SilkS") (width 0.12))
+    (fp_line (start 7.42 1.193333) (end 7.42 -0.653333) (layer "F.SilkS") (width 0.12))
+    (fp_line (start -1.92 -2.5) (end -7.92 -2.5) (layer "F.SilkS") (width 0.12))
+    (fp_line (start 7.78 3.04) (end 7.78 1.193333) (layer "F.SilkS") (width 0.12))
+    (fp_line (start -7.67 2.79) (end -7.67 -2.25) (layer "F.CrtYd") (width 0.05))
+    (fp_line (start 7.53 -2.25) (end 7.53 2.79) (layer "F.CrtYd") (width 0.05))
+    (fp_line (start -7.67 -2.25) (end 7.53 -2.25) (layer "F.CrtYd") (width 0.05))
+    (fp_line (start 7.53 2.79) (end -7.67 2.79) (layer "F.CrtYd") (width 0.05))
+    (pad "1" thru_hole rect (at 6.28 -1 270) (size 1.5 1.5) (drill 0.8) (layers *.Cu *.Mask)
       (net 15 "+3V3") (pinfunction "VCC") (pintype "power_in"))
-    (pad "2" thru_hole circle (at -3.81 1.27 270) (size 1.5 1.5) (drill 0.8) (layers *.Cu *.Mask)
+    (pad "2" thru_hole circle (at 3.74 -1 270) (size 1.5 1.5) (drill 0.8) (layers *.Cu *.Mask)
       (net 1 "GND") (pinfunction "GND") (pintype "power_in"))
-    (pad "3" thru_hole circle (at -1.27 1.27 270) (size 1.5 1.5) (drill 0.8) (layers *.Cu *.Mask)
+    (pad "3" thru_hole circle (at 1.2 -1 270) (size 1.5 1.5) (drill 0.8) (layers *.Cu *.Mask)
       (net 11 "/SFP_TX_P") (pinfunction "1") (pintype "bidirectional"))
-    (pad "4" thru_hole circle (at 1.27 1.27 270) (size 1.5 1.5) (drill 0.8) (layers *.Cu *.Mask)
+    (pad "4" thru_hole circle (at -1.34 -1 270) (size 1.5 1.5) (drill 0.8) (layers *.Cu *.Mask)
       (net 14 "/SFP_TX_N") (pinfunction "2") (pintype "bidirectional"))
-    (pad "5" thru_hole circle (at 3.81 1.27 270) (size 1.5 1.5) (drill 0.8) (layers *.Cu *.Mask)
+    (pad "5" thru_hole circle (at -3.88 -1 270) (size 1.5 1.5) (drill 0.8) (layers *.Cu *.Mask)
       (net 3 "/SFP_TX_DIS") (pinfunction "3") (pintype "bidirectional"))
-    (pad "6" thru_hole circle (at 6.35 1.27 270) (size 1.5 1.5) (drill 0.8) (layers *.Cu *.Mask)
+    (pad "6" thru_hole circle (at -6.42 -1 270) (size 1.5 1.5) (drill 0.8) (layers *.Cu *.Mask)
       (net 16 "unconnected-(U1-Pad6)") (pinfunction "4") (pintype "bidirectional+no_connect"))
-    (pad "7" thru_hole circle (at 6.35 -1.27 270) (size 1.5 1.5) (drill 0.8) (layers *.Cu *.Mask)
+    (pad "7" thru_hole circle (at -6.42 1.54 270) (size 1.5 1.5) (drill 0.8) (layers *.Cu *.Mask)
       (net 17 "unconnected-(U1-Pad7)") (pinfunction "5") (pintype "bidirectional+no_connect"))
-    (pad "8" thru_hole circle (at 3.81 -1.27 270) (size 1.5 1.5) (drill 0.8) (layers *.Cu *.Mask)
+    (pad "8" thru_hole circle (at -3.88 1.54 270) (size 1.5 1.5) (drill 0.8) (layers *.Cu *.Mask)
       (net 8 "/SFP_LOSS") (pinfunction "6") (pintype "bidirectional"))
-    (pad "9" thru_hole circle (at 1.27 -1.27 270) (size 1.5 1.5) (drill 0.8) (layers *.Cu *.Mask)
+    (pad "9" thru_hole circle (at -1.34 1.54 270) (size 1.5 1.5) (drill 0.8) (layers *.Cu *.Mask)
       (net 9 "/SFP_RX_N") (pinfunction "7") (pintype "bidirectional"))
-    (pad "10" thru_hole circle (at -1.27 -1.27 270) (size 1.5 1.5) (drill 0.8) (layers *.Cu *.Mask)
+    (pad "10" thru_hole circle (at 1.2 1.54 270) (size 1.5 1.5) (drill 0.8) (layers *.Cu *.Mask)
       (net 10 "/SFP_RX_P") (pinfunction "8") (pintype "bidirectional"))
-    (pad "11" thru_hole circle (at -3.81 -1.27 270) (size 1.5 1.5) (drill 0.8) (layers *.Cu *.Mask)
+    (pad "11" thru_hole circle (at 3.74 1.54 270) (size 1.5 1.5) (drill 0.8) (layers *.Cu *.Mask)
       (net 1 "GND") (pinfunction "GND") (pintype "power_in"))
-    (pad "12" thru_hole rect (at -6.35 -1.27 270) (size 1.5 1.5) (drill 0.8) (layers *.Cu *.Mask)
+    (pad "12" thru_hole rect (at 6.28 1.54 270) (size 1.5 1.5) (drill 0.8) (layers *.Cu *.Mask)
       (net 15 "+3V3") (pinfunction "VCC") (pintype "power_in"))
   )
@@
       (net 15 "+3V3") (pinfunction "1") (pintype "passive"))
     (pad "2" smd roundrect (at 0.485 0 180) (size 0.59 0.64) (layers "F.Cu" "F.Paste" "F.Mask") (roundrect_rratio 0.25)
-      (net 13 "Net-(J1-Pad15)") (pinfunction "2") (pintype "passive"))
+      (net 13 "Net-(C5-Pad1)") (pinfunction "2") (pintype "passive"))
     (model "${KICAD6_3DMODEL_DIR}/Inductor_SMD.3dshapes/L_0402_1005Metric.wrl"
       (offset (xyz 0 0 0))
@@
     (fp_line (start -0.5 0.25) (end -0.5 -0.25) (layer "F.Fab") (width 0.1))
     (pad "1" smd roundrect (at -0.48 0) (size 0.56 0.62) (layers "F.Cu" "F.Paste" "F.Mask") (roundrect_rratio 0.25)
-      (net 13 "Net-(J1-Pad15)") (pintype "passive"))
+      (net 13 "Net-(C5-Pad1)") (pintype "passive"))
     (pad "2" smd roundrect (at 0.48 0) (size 0.56 0.62) (layers "F.Cu" "F.Paste" "F.Mask") (roundrect_rratio 0.25)
       (net 1 "GND") (pintype "passive"))
@@
     (fp_line (start -0.5 -0.25) (end 0.5 -0.25) (layer "F.Fab") (width 0.1))
     (pad "1" smd roundrect (at -0.48 0) (size 0.56 0.62) (layers "F.Cu" "F.Paste" "F.Mask") (roundrect_rratio 0.25)
-      (net 13 "Net-(J1-Pad15)") (pintype "passive"))
+      (net 13 "Net-(C5-Pad1)") (pintype "passive"))
     (pad "2" smd roundrect (at 0.48 0) (size 0.56 0.62) (layers "F.Cu" "F.Paste" "F.Mask") (roundrect_rratio 0.25)
       (net 1 "GND") (pintype "passive"))
@@
       (net 1 "GND") (pinfunction "VeeR") (pintype "passive"))
     (pad "15" smd rect (at -2.1 0.2) (size 2 0.5) (layers "F.Cu" "F.Paste" "F.Mask")
-      (net 13 "Net-(J1-Pad15)") (pinfunction "VccR") (pintype "power_in"))
+      (net 13 "Net-(C5-Pad1)") (pinfunction "VccR") (pintype "power_in"))
     (pad "16" smd rect (at -2.1 -0.6) (size 2 0.5) (layers "F.Cu" "F.Paste" "F.Mask")
       (net 12 "Net-(C3-Pad1)") (pinfunction "VccT") (pintype "power_in"))
@@
   (gr_line (start 110.744 60.96) (end 179.832 60.96) (layer "Edge.Cuts") (width 0.1))
   (gr_line (start 179.832 60.96) (end 179.832 81.28) (layer "Edge.Cuts") (width 0.1))
+  (gr_text "https://github.com/DRubioG/pmod_sfp" (at 149.098 70.866) (layer "B.SilkS")
+    (effects (font (size 1.5 1.5) (thickness 0.3)) (justify mirror))
+  )
   (segment (start 144.018 74.93) (end 142.11 74.93) (width 0.25) (layer "F.Cu") (net 1))
   (segment (start 144.78 68.834) (end 145.666 69.72) (width 0.25) (layer "F.Cu") (net 1))

Commit message: update
Routing:
- net Net-(C3-Pad1): track 35.4 -> 34.2 mm
- net Net-(C5-Pad1): track 38.9 -> 39.9 mm
Changed lines of the file:
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@@
   )
   (setup
+    (stackup
+      (layer "F.SilkS" (type "Top Silk Screen"))
+      (layer "F.Paste" (type "Top Solder Paste"))
+      (layer "F.Mask" (type "Top Solder Mask") (thickness 0.01))
+      (layer "F.Cu" (type "copper") (thickness 0.035))
+      (layer "dielectric 1" (type "core") (thickness 1.51) (material "FR4") (epsilon_r 4.5) (loss_tangent 0.02))
+      (layer "B.Cu" (type "copper") (thickness 0.035))
+      (layer "B.Mask" (type "Bottom Solder Mask") (thickness 0.01))
+      (layer "B.Paste" (type "Bottom Solder Paste"))
+      (layer "B.SilkS" (type "Bottom Silk Screen"))
+      (copper_finish "None")
+      (dielectric_constraints no)
+    )
     (pad_to_mask_clearance 0)
     (pcbplotparams
@@
       (outputformat 1)
       (mirror false)
-      (drillshape 1)
+      (drillshape 0)
       (scaleselection 1)
-      (outputdirectory "")
+      (outputdirectory "gerber/")
     )
   )
@@
   (via (at 160.257369 70.105904) (size 0.8) (drill 0.4) (layers "F.Cu" "B.Cu") (free) (net 3))
   (via (at 147.100441 71.592853) (size 0.8) (drill 0.4) (layers "F.Cu" "B.Cu") (free) (net 3))
-  (segment (start 150.406867 71.592853) (end 152.40372 69.596) (width 0.25) (layer "B.Cu") (net 3))
   (segment (start 169.427305 74.93) (end 173.97 74.93) (width 0.25) (layer "B.Cu") (net 3))
   (segment (start 160.257369 70.105904) (end 160.471974 69.891299) (width 0.25) (layer "B.Cu") (net 3))
-  (segment (start 159.747465 69.596) (end 160.257369 70.105904) (width 0.25) (layer "B.Cu") (net 3))
+  (segment (start 148.625147 71.592853) (end 151.13 69.088) (width 0.25) (layer "B.Cu") (net 3))
+  (segment (start 151.13 69.088) (end 159.239465 69.088) (width 0.25) (layer "B.Cu") (net 3))
+  (segment (start 159.239465 69.088) (end 160.257369 70.105904) (width 0.25) (layer "B.Cu") (net 3))
+  (segment (start 147.100441 71.592853) (end 148.625147 71.592853) (width 0.25) (layer "B.Cu") (net 3))
   (segment (start 164.388604 69.891299) (end 169.427305 74.93) (width 0.25) (layer "B.Cu") (net 3))
-  (segment (start 147.100441 71.592853) (end 150.406867 71.592853) (width 0.25) (layer "B.Cu") (net 3))
   (segment (start 160.471974 69.891299) (end 164.388604 69.891299) (width 0.25) (layer "B.Cu") (net 3))
-  (segment (start 152.40372 69.596) (end 159.747465 69.596) (width 0.25) (layer "B.Cu") (net 3))
   (segment (start 142.1 72.52) (end 144.396 72.52) (width 0.25) (layer "F.Cu") (net 7))
   (segment (start 144.396 72.52) (end 144.526 72.39) (width 0.25) (layer "F.Cu") (net 7))
@@
   (via (at 166.878 66.548) (size 0.8) (drill 0.4) (layers "F.Cu" "B.Cu") (net 12))
   (via (at 144.78 70.358) (size 0.8) (drill 0.4) (layers "F.Cu" "B.Cu") (free) (net 12))
-  (segment (start 147.066 67.554695) (end 147.066 68.072) (width 0.25) (layer "B.Cu") (net 12))
-  (segment (start 153.89428 66.294) (end 152.84528 65.245) (width 0.25) (layer "B.Cu") (net 12))
-  (segment (start 152.84528 65.245) (end 149.976305 65.245) (width 0.25) (layer "B.Cu") (net 12))
+  (segment (start 166.624 66.294) (end 153.89428 66.294) (width 0.25) (layer "B.Cu") (net 12))
+  (segment (start 153.89428 66.294) (end 153.475 66.71328) (width 0.25) (layer "B.Cu") (net 12))
+  (segment (start 152.67628 67.564) (end 147.574 67.564) (width 0.25) (layer "B.Cu") (net 12))
+  (segment (start 147.574 67.564) (end 144.78 70.358) (width 0.25) (layer "B.Cu") (net 12))
+  (segment (start 153.475 66.76528) (end 152.67628 67.564) (width 0.25) (layer "B.Cu") (net 12))
   (segment (start 166.878 66.548) (end 166.624 66.294) (width 0.25) (layer "B.Cu") (net 12))
-  (segment (start 166.624 66.294) (end 153.89428 66.294) (width 0.25) (layer "B.Cu") (net 12))
-  (segment (start 147.066 68.072) (end 144.78 70.358) (width 0.25) (layer "B.Cu") (net 12))
-  (segment (start 148.035695 66.585) (end 147.066 67.554695) (width 0.25) (layer "B.Cu") (net 12))
-  (segment (start 148.636305 66.585) (end 148.035695 66.585) (width 0.25) (layer "B.Cu") (net 12))
-  (segment (start 149.976305 65.245) (end 148.636305 66.585) (width 0.25) (layer "B.Cu") (net 12))
+  (segment (start 153.475 66.71328) (end 153.475 66.76528) (width 0.25) (layer "B.Cu") (net 12))
   (segment (start 165.862 69.85) (end 165.354 70.358) (width 0.25) (layer "F.Cu") (net 13))
   (segment (start 164.592 70.358) (end 164.346598 70.358) (width 0.25) (layer "F.Cu") (net 13))
@@
   (via (at 164.088299 70.616299) (size 0.8) (drill 0.4) (layers "F.Cu" "B.Cu") (free) (net 13))
   (via (at 147.574 72.644) (size 0.8) (drill 0.4) (layers "F.Cu" "B.Cu") (free) (net 13))
-  (segment (start 162.060598 72.644) (end 147.574 72.644) (width 0.25) (layer "B.Cu") (net 13))
-  (segment (start 164.088299 70.616299) (end 162.060598 72.644) (width 0.25) (layer "B.Cu") (net 13))
+  (segment (start 158.97616 69.85) (end 151.258396 69.85) (width 0.25) (layer "B.Cu") (net 13))
+  (segment (start 161.030578 70.358) (end 160.557674 70.830904) (width 0.25) (layer "B.Cu") (net 13))
+  (segment (start 149.065543 72.042853) (end 148.175147 72.042853) (width 0.25) (layer "B.Cu") (net 13))
+  (segment (start 148.175147 72.042853) (end 147.574 72.644) (width 0.25) (layer "B.Cu") (net 13))
+  (segment (start 159.957064 70.830904) (end 158.97616 69.85) (width 0.25) (layer "B.Cu") (net 13))
+  (segment (start 160.557674 70.830904) (end 159.957064 70.830904) (width 0.25) (layer "B.Cu") (net 13))
+  (segment (start 164.088299 70.616299) (end 163.83 70.358) (width 0.25) (layer "B.Cu") (net 13))
+  (segment (start 151.258396 69.85) (end 149.065543 72.042853) (width 0.25) (layer "B.Cu") (net 13))
+  (segment (start 163.83 70.358) (end 161.030578 70.358) (width 0.25) (layer "B.Cu") (net 13))
   (segment (start 160.02 71.374) (end 168.91 71.374) (width 0.2) (layer "F.Cu") (net 14))
   (segment (start 156.766 68.12) (end 160.02 71.374) (width 0.2) (layer "F.Cu") (net 14))
